File: hardware/Raspberry Pi temperature management hat.kicad_sch (KiCad schematic)
At the start: 28 parts, among them J1 Screw Terminal x3, J2 Screw Terminal x2, J3 OX40HAT, Q1 S8050, U1 MIC5225-3.3, U2 MAX31865, U3 LTV-817S

Commit message: PCB board V2
Parts:
- removed D1, D2, D3: 1N4148W, Diode_SMD:D_0603_1608Metric_Pad1.05x0.95mm_HandSolder, symbol Diode:1N4148W
- removed D5: S1MFL, Diode_SMD:D_SOD-123F, symbol Diode:US1M
- removed H3, H4: 3mm_Mounting_Hole, project_footprints:NPTH_3mm_ID, symbol Mechanical:MountingHole
- removed R1, R2: 10k, Resistor_SMD:R_0603_1608Metric_Pad0.98x0.95mm_HandSolder, symbol Device:R
- added D2, D4: LL4148, Diode_SMD:D_MiniMELF_Handsoldering, symbol Diode:LL4148
- added D3: LED, LED_SMD:LED_0603_1608Metric_Pad1.05x0.95mm_HandSolder, symbol Device:LED
- added H3, H4: MountingHole_Pad, MountingHole:MountingHole_3mm_Pad, symbol Mechanical:MountingHole_Pad
- added J2: Screw Terminal x2, TerminalBlock_MetzConnect:TerminalBlock_MetzConnect_Type055_RT01502HDWU_1x02_P5.00mm_Horizontal, symbol Connector:Screw_Terminal_01x02
- added Q2: S8050, Package_TO_SOT_SMD:SOT-23_Handsoldering, symbol Transistor_BJT:S8050
- added R4: 510, Resistor_SMD:R_0603_1608Metric_Pad0.98x0.95mm_HandSolder, symbol Device:R
- added U2: LTV-817S, Package_DIP:SMDIP-4_W9.53mm, symbol Isolator:LTV-817S
- F1: footprint Fuse:Fuse_0402_1005Metric_Pad0.77x0.64mm_HandSolder -> Fuse:Fuse_0603_1608Metric_Pad1.05x0.95mm_HandSolder
- H1, H2: value 3mm_Mounting_Hole -> MountingHole; footprint project_footprints:NPTH_3mm_ID -> MountingHole:MountingHole_3mm
- J1: renamed from J2; footprint TerminalBlock_TE-Connectivity:TerminalBlock_TE_282834-2_1x02_P2.54mm_Horizontal -> TerminalBlock_MetzConnect:TerminalBlock_MetzConnect_Type055_RT01502HDWU_1x02_P5.00mm_Horizontal
- J3: renamed from J1; footprint TerminalBlock_TE-Connectivity:TerminalBlock_TE_282834-3_1x03_P2.54mm_Horizontal -> TerminalBlock_MetzConnect:TerminalBlock_MetzConnect_Type055_RT01503HDWU_1x03_P5.00mm_Horizontal
- R3: value 10k -> 180
- renumbered C3 to C1, C1 to C2, C4 to C3, C2 to C4, D4 to D1, J3 to J4, R5 to R1, R6 to R2, R4 to R5, U3 to U1, U1 to U3, U2 to U4
Connections:
- net +5V: now also D2.1 (K), D4.1 (K), J2.1 (Pin_1), U2.4
- net CS: now also U4.13 (CS)
- net GND: now also J4.39 (GND), D3.1 (K), H3.1, H4.1, Q2.1 (E); no longer J4.9 (GND)
- net SCLK: now also U4.12 (SCLK)
- net SDI: now also U4.11 (SDI)
- net VDD: no longer R3.1
- net HET: now reaches J4.11 (GPIO17)
- net HET: now also R1.2
- net FAN: now reaches J4.15 (GPIO22)
- net FAN: now also R3.2
- net at J1.2 (Pin_2), Q1.3 (C): now also D2.2 (A)
- net at U4.5 (FORCE+), U4.6 (FORCE2): now also J3.3 (Pin_3); no longer J3.1 (Pin_1)
- net at C5.2, U4.8 (RTDIN-), U4.9 (FORCE-): now also J3.1 (Pin_1); no longer J3.3 (Pin_3)
- net REL: no longer names the net of J4.27 (GPIO00)
- net REL: no longer R1.2
- new net: R3.1, U2.1
- new net: R4.1, U2.3
- new net: Q2.2 (B), R4.2
- new net: D3.2 (A), U2.2
- new net: D4.2 (A), J2.2 (Pin_2), Q2.3 (C)
Other:
- note added: "Fan relay"
- note added: "Heating relay"
- note added: "MAX31865 3.3V voltage stabilizer"
- note added: "MAX31865 IC configured for 3 wire temperature sensor"
- note added: "Raspberry Pi 4B pin socket"
- moved on the sheet: C1, C2, C3, C4, C5, F1, J3, R5, U3, U4

Commit message: final version of V2 board with gerber files
Parts:
- D2, D4: footprint Diode_SMD:D_MiniMELF_Handsoldering -> Diode_SMD:D_MiniMELF
- J1, J2: footprint TerminalBlock_MetzConnect:TerminalBlock_MetzConnect_Type055_RT01502HDWU_1x02_P5.00mm_Horizontal -> TerminalBlock_Phoenix:TerminalBlock_Phoenix_PT-1,5-2-3.5-H_1x02_P3.50mm_Horizontal
- J3: footprint TerminalBlock_MetzConnect:TerminalBlock_MetzConnect_Type055_RT01503HDWU_1x03_P5.00mm_Horizontal -> TerminalBlock_Phoenix:TerminalBlock_Phoenix_PT-1,5-3-3.5-H_1x03_P3.50mm_Horizontal
Connections:
- net +5V: now also J1.2 (Pin_2), J2.2 (Pin_2); no longer J1.1 (Pin_1), J2.1 (Pin_1)
- net at D2.2 (A), Q1.3 (C): now also J1.1 (Pin_1); no longer J1.2 (Pin_2)
- net at U4.5 (FORCE+), U4.6 (FORCE2): now also J3.1 (Pin_1); no longer J3.3 (Pin_3)
- net at C5.2, U4.8 (RTDIN-), U4.9 (FORCE-): now also J3.3 (Pin_3); no longer J3.1 (Pin_1)
- net at D4.2 (A), Q2.3 (C): now also J2.1 (Pin_1); no longer J2.2 (Pin_2)
Changed lines of the file:
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@@
     (title "Raspberry Pi temperature management hat")
     (date "2022-06-14")
-    (rev "V1")
+    (rev "V2")
   )
   (junction (at 130.81 63.5) (diameter 0) (color 0 0 0 0)
@@
       (effects (font (size 1.27 1.27)) (justify left))
     )
-    (property "Footprint" "Diode_SMD:D_MiniMELF_Handsoldering" (id 2) (at 240.665 114.3 0)
+    (property "Footprint" "Diode_SMD:D_MiniMELF" (id 2) (at 240.665 114.3 0)
       (effects (font (size 1.27 1.27)) hide)
     )
@@
     (pin "2")
   )
-  (symbol (lib_id "Connector:Screw_Terminal_01x02") (at 254 38.1 0) (unit 1)
-    (in_bom yes) (on_board yes) (fields_autoplaced)
-    (property "Reference" "J1" (id 0) (at 256.54 38.0999 0)
-      (effects (font (size 1.27 1.27)) (justify left))
-    )
-    (property "Value" "Screw Terminal x2" (id 1) (at 256.54 40.6399 0)
-      (effects (font (size 1.27 1.27)) (justify left))
-    )
-    (property "Footprint" "TerminalBlock_MetzConnect:TerminalBlock_MetzConnect_Type055_RT01502HDWU_1x02_P5.00mm_Horizontal" (id 2) (at 254 34.925 0)
-      (effects (font (size 1.27 1.27)) hide)
-    )
-    (property "Datasheet" "~" (id 3) (at 254 38.1 0)
-      (effects (font (size 1.27 1.27)) hide)
-    )
-    (pin "1")
-    (pin "2")
-  )
-  (symbol (lib_id "Connector:Screw_Terminal_01x03") (at 168.91 93.98 0) (mirror x) (unit 1)
-    (in_bom yes) (on_board yes) (fields_autoplaced)
-    (property "Reference" "J3" (id 0) (at 168.91 85.09 0))
-    (property "Value" "Screw Terminal x3" (id 1) (at 168.91 87.63 0))
-    (property "Footprint" "TerminalBlock_MetzConnect:TerminalBlock_MetzConnect_Type055_RT01503HDWU_1x03_P5.00mm_Horizontal" (id 2) (at 168.91 93.98 0)
+  (symbol (lib_id "Connector:Screw_Terminal_01x02") (at 254 40.64 0) (mirror x) (unit 1)
+    (in_bom yes) (on_board yes)
+    (property "Reference" "J1" (id 0) (at 257.81 38.1 0))
+    (property "Value" "Screw Terminal x2" (id 1) (at 265.43 40.64 0))
+    (property "Footprint" "TerminalBlock_Phoenix:TerminalBlock_Phoenix_PT-1,5-2-3.5-H_1x02_P3.50mm_Horizontal" (id 2) (at 254 43.815 0)
+      (effects (font (size 1.27 1.27)) hide)
+    )
+    (property "Datasheet" "~" (id 3) (at 254 40.64 0)
+      (effects (font (size 1.27 1.27)) hide)
+    )
+    (pin "1")
+    (pin "2")
+  )
+  (symbol (lib_id "Connector:Screw_Terminal_01x03") (at 168.91 93.98 0) (unit 1)
+    (in_bom yes) (on_board yes) (fields_autoplaced)
+    (property "Reference" "J3" (id 0) (at 171.45 92.7099 0)
+      (effects (font (size 1.27 1.27)) (justify left))
+    )
+    (property "Value" "Screw Terminal x3" (id 1) (at 171.45 95.2499 0)
+      (effects (font (size 1.27 1.27)) (justify left))
+    )
+    (property "Footprint" "TerminalBlock_Phoenix:TerminalBlock_Phoenix_PT-1,5-3-3.5-H_1x03_P3.50mm_Horizontal" (id 2) (at 168.91 93.98 0)
       (effects (font (size 1.27 1.27)) hide)
     )
@@
       (effects (font (size 1.27 1.27)) (justify left))
     )
-    (property "Footprint" "Diode_SMD:D_MiniMELF_Handsoldering" (id 2) (at 239.395 39.37 0)
+    (property "Footprint" "Diode_SMD:D_MiniMELF" (id 2) (at 239.395 39.37 0)
       (effects (font (size 1.27 1.27)) hide)
     )
@@
     (pin "1")
   )
-  (symbol (lib_id "Connector:Screw_Terminal_01x02") (at 255.27 113.03 0) (unit 1)
-    (in_bom yes) (on_board yes) (fields_autoplaced)
-    (property "Reference" "J2" (id 0) (at 257.81 113.0299 0)
-      (effects (font (size 1.27 1.27)) (justify left))
-    )
-    (property "Value" "Screw Terminal x2" (id 1) (at 257.81 115.5699 0)
-      (effects (font (size 1.27 1.27)) (justify left))
-    )
-    (property "Footprint" "TerminalBlock_MetzConnect:TerminalBlock_MetzConnect_Type055_RT01502HDWU_1x02_P5.00mm_Horizontal" (id 2) (at 255.27 109.855 0)
-      (effects (font (size 1.27 1.27)) hide)
-    )
-    (property "Datasheet" "~" (id 3) (at 255.27 113.03 0)
+  (symbol (lib_id "Connector:Screw_Terminal_01x02") (at 255.27 115.57 0) (mirror x) (unit 1)
+    (in_bom yes) (on_board yes)
+    (property "Reference" "J2" (id 0) (at 259.08 113.03 0))
+    (property "Value" "Screw Terminal x2" (id 1) (at 266.7 115.57 0))
+    (property "Footprint" "TerminalBlock_Phoenix:TerminalBlock_Phoenix_PT-1,5-2-3.5-H_1x02_P3.50mm_Horizontal" (id 2) (at 255.27 118.745 0)
+      (effects (font (size 1.27 1.27)) hide)
+    )
+    (property "Datasheet" "~" (id 3) (at 255.27 115.57 0)
       (effects (font (size 1.27 1.27)) hide)
     )
@@
     )
     (path "/f3c363ba-a7e3-496d-ac78-b86b35cbcafd"
-      (reference "D2") (unit 1) (value "LL4148") (footprint "Diode_SMD:D_MiniMELF_Handsoldering")
+      (reference "D2") (unit 1) (value "LL4148") (footprint "Diode_SMD:D_MiniMELF")
     )
     (path "/1fb47b55-2309-4bbf-abff-72b25a4d0f9b"
@@
     )
     (path "/d8ba865b-fbf1-426e-8a95-c2dad77c2ea8"
-      (reference "D4") (unit 1) (value "LL4148") (footprint "Diode_SMD:D_MiniMELF_Handsoldering")
+      (reference "D4") (unit 1) (value "LL4148") (footprint "Diode_SMD:D_MiniMELF")
     )
     (path "/32a2edc4-7913-4ae5-b3c7-8f26c88b8b9d"
@@
     )
     (path "/e309bf98-7bac-42d5-8a1d-a65a8f9fcd63"
-      (reference "J1") (unit 1) (value "Screw Terminal x2") (footprint "TerminalBlock_MetzConnect:TerminalBlock_MetzConnect_Type055_RT01502HDWU_1x02_P5.00mm_Horizontal")
+      (reference "J1") (unit 1) (value "Screw Terminal x2") (footprint "TerminalBlock_Phoenix:TerminalBlock_Phoenix_PT-1,5-2-3.5-H_1x02_P3.50mm_Horizontal")
     )
     (path "/f764b93c-4f58-425a-8a99-562154c17b64"
-      (reference "J2") (unit 1) (value "Screw Terminal x2") (footprint "TerminalBlock_MetzConnect:TerminalBlock_MetzConnect_Type055_RT01502HDWU_1x02_P5.00mm_Horizontal")
+      (reference "J2") (unit 1) (value "Screw Terminal x2") (footprint "TerminalBlock_Phoenix:TerminalBlock_Phoenix_PT-1,5-2-3.5-H_1x02_P3.50mm_Horizontal")
     )
     (path "/e7dbbbf1-8a33-4a55-b7b5-f86d84ed24f1"
-      (reference "J3") (unit 1) (value "Screw Terminal x3") (footprint "TerminalBlock_MetzConnect:TerminalBlock_MetzConnect_Type055_RT01503HDWU_1x03_P5.00mm_Horizontal")
+      (reference "J3") (unit 1) (value "Screw Terminal x3") (footprint "TerminalBlock_Phoenix:TerminalBlock_Phoenix_PT-1,5-3-3.5-H_1x03_P3.50mm_Horizontal")
     )
     (path "/0593dc7a-b268-4003-a428-ec8b71b7ef13"

Commit message: stencil gerber file added
Parts:
- U3: value MIC5225-3.3 -> MIC5245-3.3
Changed lines of the file:
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@@
     (in_bom yes) (on_board yes) (fields_autoplaced)
     (property "Reference" "U3" (id 0) (at 59.69 33.02 0))
-    (property "Value" "MIC5225-3.3" (id 1) (at 59.69 35.56 0))
+    (property "Value" "MIC5245-3.3" (id 1) (at 59.69 35.56 0))
     (property "Footprint" "Package_TO_SOT_SMD:SOT-23-5_HandSoldering" (id 2) (at 59.69 48.26 0)
       (effects (font (size 1.27 1.27)) hide)
@@
     )
     (path "/b1f6acb2-8a8a-4c61-a848-32dbc95b6268"
-      (reference "U3") (unit 1) (value "MIC5225-3.3") (footprint "Package_TO_SOT_SMD:SOT-23-5_HandSoldering")
+      (reference "U3") (unit 1) (value "MIC5245-3.3") (footprint "Package_TO_SOT_SMD:SOT-23-5_HandSoldering")
     )
     (path "/a26cd88b-81d1-4769-9b71-447258a65dc5"
